File: pcb/rusty-collars-p4-carrier.kicad_pcb (KiCad board)
At the start: 2 copper layers, 85 x 56 mm, 12 parts, among them J1 ESP32_P4_VBUS_SIDE, J2 ESP32_P4_GPIO54_SIDE, J3 TX_433MHZ, J4 RX_433MHZ

Commit message: pcb
Parts:
- added ?: , , F.Cu at (132.3, 122.7)
- added ?: , , F.Cu at (119.0, 101.3)
Routing:
- net /+3V3: track 81.1 -> 108.7 mm
- net /GND: track 229.3 -> 235.0 mm
- net /GPIO17: track 74.2 -> 79.5 mm

Commit message: reproducible toolchain
Parts:
- moved ? 7.62 mm to (111.4, 101.3)
- moved D1 7.62 mm to (174.9, 86.0)
- moved D2 7.62 mm to (174.9, 124.0)
- moved J1 7.62 mm to (116.8, 96.1)
- moved J2 7.62 mm to (116.8, 113.9)
- moved J3 7.62 mm to (137.1, 82.0)
- moved J4 7.62 mm to (137.1, 128.0)
- moved R1 7.62 mm to (159.4, 86.0)
- moved R2 7.62 mm to (160.3, 124.0)
- moved ? 7.62 mm to (124.7, 122.7)
Routing:
- net /+3V3: track 108.7 -> 98.9 mm
